File: pcbOrthoLinear/LetsSplit256o.sch (KiCad schematic (older format))
At the start: 62 parts, among them U1 ProMicro

Commit message: Generate geber
Parts:
- U1: symbol void_keeb-cache:promicro_ProMicro -> LetsSplit256-rescue:promicro_ProMicro-void_keeb-cache
Changed lines of the file:
@@
 $EndDescr
 $Comp
-L void_keeb-cache:promicro_ProMicro U1
+L LetsSplit256-rescue:promicro_ProMicro-void_keeb-cache U1
 U 1 1 5BB733A3
 P 7300 3500
